File: gnss_antenna_pcb/gnss_antenna_pcb.kicad_sch (KiCad schematic)
At the start: 32 parts, among them J1 uFL, J2 Conn_Coaxial_Power, Q1 BFP640FESD, U1 NCV8163ASN330T1G

Commit message: Update PCB
Connections:
- net at R1.2, R2.2: now also MW1.3 (Out); no longer MW1.4 (Match)
- net at C1.1: now also MW1.4 (Match); no longer MW1.3 (Out)
Other:
- note added: "Between the antenna and the amplifier there should be a matching transmission line, a microstrip line with 1,485 mm width and 26,5 mm length. This is required for impedance matching of the amplifier."
- note added: "This assembly of a coaxial connector and capacitor is to allow the creation of a test point for the RF path. Being able to switch the mounting position of the capacitor and hence shift between measuring the antenna or the amplifier."
- note removed: "Between the antenna and the amplifier there should be a matching transmission line, a microstrip line with 2 mm width and 27 mm length. This is required otherwise the amplifier will not perform as expected."
- note removed: "This assembly of a coaxial connector and capacitor is actually to be able to create a test point for the RF path. Being able to switch the mounting position of the capacitor and hence shift between measuring the antenna or the amplifier."
- moved on the sheet: AE1, MW1, R1, R2
